File: VCA_Panner/untitled.kicad_sch (KiCad schematic)
At the start: 43 parts, among them U1 TL074, U2 TL074, U4 TL074

Commit message: finished schematic
Parts:
- removed C1, C10, C11, C3, C8, C9: 47pF, symbol Device:C
- removed D2, D4: D, symbol Device:D
- removed R1, R19, R21, R24: 51k, symbol Device:R
- removed R10, R18, R5: 99k, symbol Device:R
- removed R11, R12, R13, R17, R4: 1k, symbol Device:R
- removed R14, R20, R25, R26, R7, R8: 100k, symbol Device:R
- removed R15, R16: 330k, symbol Device:R
- removed R2, R3: 4.7M, symbol Device:R
- removed R22, R27: 10k, symbol Device:R
- removed R23, R28: 400k, symbol Device:R
- removed R6: 99900, symbol Device:R
- removed R9: 100, symbol Device:R
- removed U1, U2, U4: TL074, symbol Amplifier_Operational:TL074
- removed V1, V4: VSIN, symbol Simulation_SPICE:VSIN
- removed V2: 12, symbol Simulation_SPICE:VDC
- removed V3: -12, symbol Simulation_SPICE:VDC
