File: VCO-3340/VCO-3340.kicad_pcb (KiCad board)
At the start: 2 copper layers, 48.8 x 110 mm, 102 parts, among them J1 1V/oct in, J10 SIN_OUT, J2 cv_mod_in, J3 pwm_mod_in, J4 fm_mod_in, J5 sync_in, J6 Eurorack_Power_10pin_Unshroud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, J7 PULSE_OUT, J8 SAW_OUT, J9 TRI_OUT, SW1 PWM SRC SEL, SW2 SYNC MODE, U1 AS3340, U2 LM337L_TO92, U3 L78L05_TO92, U4 TL074

Commit message: feitw bugfixes
Parts:
- D1: footprint Diode_SMD:D_SOD-323F -> Diode_THT:D_DO-41_SOD81_P2.54mm_Vertical_AnodeUp; moved to B.Cu
- D2: footprint Diode_SMD:D_SOD-323F -> Diode_THT:D_DO-41_SOD81_P2.54mm_Vertical_AnodeUp
- R24: footprint Resistor_SMD:R_0805_2012Metric_Pad1.20x1.40mm_HandSolder -> Resistor_THT:R_Axial_DIN0204_L3.6mm_D1.6mm_P1.90mm_Vertical; moved to B.Cu
- R25: footprint Resistor_SMD:R_0805_2012Metric_Pad1.20x1.40mm_HandSolder -> Resistor_THT:R_Axial_DIN0204_L3.6mm_D1.6mm_P1.90mm_Vertical
- U2: value LM337L_TO92 -> LM337L_SO8; footprint Package_SO:SO-8_3.9x4.9mm_P1.27mm -> Package_SO:SOIC-8_3.9x4.9mm_P1.27mm
- moved D2 8.76 mm to (53.0, 35.9)
- moved D1 7.60 mm to (38.1, 49.2), turned to 90 degrees
- moved R25 5.68 mm to (38.0, 41.6)
- moved R24 2.54 mm to (38.4, 54.7)
- moved C14 2.20 mm to (34.5, 55.0)
Connections:
- C12 pad 1: -7V5 -> GND
- C12 pad 2: GND -> -7V5
- U2 pad 1: Net-(U2-ADJ) -> -7V5
- U2 pad 2: -7V5 -> -12V
- U2 pad 4: (no net) -> Net-(U2-ADJ)
- U2 pad 5: (no net) -> unconnected-(U2-NC-Pad5)
- U2 pad 6: (no net) -> -12V
- U2 pad 7: (no net) -> -12V
- U2 pad 8: (no net) -> unconnected-(U2-NC-Pad8)
Routing:
- net Net-(D2-A): track 2.46 -> 14.8 mm
- net Net-(U2-ADJ): track 5.02 -> 12.4 mm, vias 0 -> 2
- net Net-(D2-K): track 6.85 -> 12.7 mm
- net -12V: track 96.5 -> 102.2 mm, vias 1 -> 3
- net -7V5: track 93.8 -> 97.9 mm, vias 0 -> 1
- net +12V: track 135.6 -> 132.6 mm
- net Net-(D1-A): track 6.75 -> 9.23 mm
- net Net-(D1-K): track 2.21 -> 3.75 mm
- net Net-(U1-VFCI): track 127.6 -> 128.6 mm
- net GND: vias 74 -> 76
