File: VCO-3340/VCO-3340.kicad_sch (KiCad schematic)
At the start: 102 parts, among them J1 1V/oct in, J10 SIN_OUT, J2 cv_mod_in, J3 pwm_mod_in, J4 fm_mod_in, J5 sync_in, J6 Eurorack_Power_10pin_Unshroud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, J7 PULSE_OUT, J8 SAW_OUT, J9 TRI_OUT, SW1 PWM SRC SEL, SW2 SYNC MODE, U1 AS3340, U2 LM337L_SO8, U3 L78L05_TO92, U4 TL074

Commit message: bugfixes fpr 3340
Parts:
- R6: value 100k -> 1M8
- RV2, RV3, RV5, RV7, RV8, RV9: value 100k -> B100k
Changed lines of the file:
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@@
 			)
 		)
-		(property "Value" "100k"
+		(property "Value" "B100k"
 			(at 38.862 103.632 0)
 			(effects
@@
 			)
 		)
-		(property "Value" "100k"
+		(property "Value" "1M8"
 			(at 50.8 39.37 90)
 			(effects
@@
 			)
 		)
-		(property "Value" "100k"
+		(property "Value" "B100k"
 			(at 38.862 131.572 0)
 			(effects
@@
 			)
 		)
-		(property "Value" "100k"
+		(property "Value" "B100k"
 			(at 36.322 75.692 0)
 			(effects
@@
 			)
 		)
-		(property "Value" "100k"
+		(property "Value" "B100k"
 			(at 35.56 25.4001 0)
 			(effects
@@
 			)
 		)
-		(property "Value" "100k"
+		(property "Value" "B100k"
 			(at 35.56 41.9101 0)
 			(effects
@@
 			)
 		)
-		(property "Value" "100k"
+		(property "Value" "B100k"
 			(at 76.708 131.572 0)
 			(effects
