File: VCO-3340/VCO-3340.kicad_sch (KiCad schematic)
At the start: 102 parts, among them J1 1V/oct in, J10 SIN_OUT, J2 cv_mod_in, J3 pwm_mod_in, J4 fm_mod_in, J5 sync_in, J6 Eurorack_Power_10pin_Unshroud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, J7 PULSE_OUT, J8 SAW_OUT, J9 TRI_OUT, SW1 PWM SRC SEL, SW2 SYNC MODE, U1 AS3340, U2 LM337L_TO92, U3 L78L05_TO92, U4 TL074

Commit message: feitw bugfixes
Parts:
- removed U2: LM337L_TO92, Package_SO:SO-8_3.9x4.9mm_P1.27mm, symbol Regulator_Linear:LM337L_TO92
- added U2: LM337L_SO8, Package_SO:SOIC-8_3.9x4.9mm_P1.27mm, symbol Regulator_Linear:LM337L_SO8
- D1, D2: footprint Diode_SMD:D_SOD-323F -> Diode_THT:D_DO-41_SOD81_P2.54mm_Vertical_AnodeUp
- R24, R25: footprint Resistor_SMD:R_0805_2012Metric_Pad1.20x1.40mm_HandSolder -> Resistor_THT:R_Axial_DIN0204_L3.6mm_D1.6mm_P1.90mm_Vertical
Connections:
- net -12V: now also U2.2 (VI), U2.3 (VI), U2.6 (VI), U2.7 (VI)
- net -7V5: now also C12.2, U2.1 (VO); no longer C12.1
- net GND: now also C12.1; no longer C12.2
- net at R22.1, R23.1: now also U2.4 (ADJ)
Other:
- company: (none) -> Clandestine Circutry
- title: (none) -> 3340 VCO
- moved on the sheet: C12
Changed lines of the file:
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@@
 	(generator_version "8.0")
 	(paper "A4")
+	(title_block
+		(title "3340 VCO")
+		(date "2024-06-12")
+		(rev "2")
+		(company "Clandestine Circutry")
+	)
 	(junction
 		(at 128.27 154.94)
@@
 	)
 	(symbol
-		(lib_id "Regulator_Linear:LM337L_TO92")
-		(at 41.91 171.45 0)
-		(mirror x)
-		(unit 1)
-		(exclude_from_sim no)
-		(in_bom yes)
-		(on_board yes)
-		(dnp no)
-		(property "Reference" "U2"
-			(at 41.91 165.1 0)
-			(effects
-				(font
-					(size 1.27 1.27)
-				)
-			)
-		)
-		(property "Value" "LM337L_TO92"
-			(at 41.91 167.64 0)
-			(effects
-				(font
-					(size 1.27 1.27)
-				)
-			)
-		)
-		(property "Footprint" "Package_SO:SO-8_3.9x4.9mm_P1.27mm"
-			(at 41.91 166.37 0)
-			(effects
-				(font
-					(size 1.27 1.27)
-					(italic yes)
-				)
-				(hide yes)
-			)
-		)
-		(property "Datasheet" "http://www.ti.com/lit/ds/symlink/lm337l.pdf"
-			(at 41.91 171.45 0)
-			(effects
-				(font
-					(size 1.27 1.27)
-				)
-				(hide yes)
-			)
-		)
-		(property "Description" "Negative 100mA 35V Adjustable Linear Regulator, TO-92"
-			(at 41.91 171.45 0)
-			(effects
-				(font
-					(size 1.27 1.27)
-				)
-				(hide yes)
-			)
-		)
-		(pin "1"
-		)
-		(pin "3"
-		)
-		(pin "2"
-		)
-		(instances
-			(project "VCO-3340"
-				(path "/83927a7b-f31e-475f-ac55-cd2bf2a0e341"
-					(reference "U2")
-					(unit 1)
-				)
-			)
-		)
-	)
-	(symbol
 		(lib_id "Connector_Audio:AudioJack2_SwitchT")
 		(at 24.13 102.87 0)
@@
 			)
 		)
-		(property "Footprint" "Diode_SMD:D_SOD-323F"
+		(property "Footprint" "Diode_THT:D_DO-41_SOD81_P2.54mm_Vertical_AnodeUp"
 			(at 116.84 140.335 0)
 			(effects
@@
 	)
 	(symbol
+		(lib_id "Regulator_Linear:LM337L_SO8")
+		(at 41.91 171.45 0)
+		(mirror x)
+		(unit 1)
+		(exclude_from_sim no)
+		(in_bom yes)
+		(on_board yes)
+		(dnp no)
+		(fields_autoplaced yes)
+		(property "Reference" "U2"
+			(at 41.91 165.1 0)
+			(effects
+				(font
+					(size 1.27 1.27)
+				)
+			)
+		)
+		(property "Value" "LM337L_SO8"
+			(at 41.91 167.64 0)
+			(effects
+				(font
+					(size 1.27 1.27)
+				)
+			)
+		)
+		(property "Footprint" "Package_SO:SOIC-8_3.9x4.9mm_P1.27mm"
+			(at 41.91 166.37 0)
+			(effects
+				(font
+					(size 1.27 1.27)
+					(italic yes)
+				)
+				(hide yes)
+			)
+		)
+		(property "Datasheet" "http://www.ti.com/lit/ds/symlink/lm337l.pdf"
+			(at 41.91 171.45 0)
+			(effects
+				(font
+					(size 1.27 1.27)
+				)
+				(hide yes)
+			)
+		)
+		(property "Description" "100mA 35V Adjustable Negative Linear Regulator, SO-8"
+			(at 41.91 171.45 0)
+			(effects
+				(font
+					(size 1.27 1.27)
+				)
+				(hide yes)
+			)
+		)
+		(pin "1"
+		)
+		(pin "7"
+		)
+		(pin "2"
+		)
+		(pin "6"
+		)
+		(pin "4"
+		)
+		(pin "3"
+		)
+		(pin "5"
+		)
+		(pin "8"
+		)
+		(instances
+			(project "VCO-3340"
+				(path "/83927a7b-f31e-475f-ac55-cd2bf2a0e341"
+					(reference "U2")
+					(unit 1)
+				)
+			)
+		)
+	)
+	(symbol
 		(lib_id "power:+5V")
 		(at 114.3 172.72 0)
@@
 			)
 		)
-		(property "Footprint" "Resistor_SMD:R_0805_2012Metric_Pad1.20x1.40mm_HandSolder"
+		(property "Footprint" "Resistor_THT:R_Axial_DIN0204_L3.6mm_D1.6mm_P1.90mm_Vertical"
 			(at 124.46 156.718 90)
 			(effects
@@
 			)
 		)
-		(property "Footprint" "Resistor_SMD:R_0805_2012Metric_Pad1.20x1.40mm_HandSolder"
+		(property "Footprint" "Resistor_THT:R_Axial_DIN0204_L3.6mm_D1.6mm_P1.90mm_Vertical"
 			(at 124.46 143.002 90)
 			(effects
@@
 			)
 		)
-		(property "Footprint" "Diode_SMD:D_SOD-323F"
+		(property "Footprint" "Diode_THT:D_DO-41_SOD81_P2.54mm_Vertical_AnodeUp"
 			(at 116.84 159.385 0)
 			(effects
@@
 	(symbol
 		(lib_id "Device:C_Polarized")
-		(at 74.93 177.8 0)
+		(at 74.93 177.8 180)
 		(unit 1)
 		(exclude_from_sim no)
@@
 		(fields_autoplaced yes)
 		(property "Reference" "C12"
-			(at 78.74 175.6409 0)
+			(at 78.74 177.4189 0)
 			(effects
 				(font
 					(size 1.27 1.27)
 				)
-				(justify left)
+				(justify right)
 			)
 		)
 		(property "Value" "10uF/25V"
-			(at 78.74 178.1809 0)
+			(at 78.74 179.9589 0)
 			(effects
 				(font
 					(size 1.27 1.27)
 				)
-				(justify left)
+				(justify right)
 			)
 		)
 		(property "Footprint" "Capacitor_THT:CP_Radial_D4.0mm_P2.00mm"
-			(at 75.8952 181.61 0)
+			(at 73.9648 173.99 0)
 			(effects
 				(font

Commit message: fixed some things
Parts:
- R6: value 100k -> 1M8
Changed lines of the file:
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@@
 			)
 		)
-		(property "Value" "100k"
+		(property "Value" "1M8"
 			(at 50.8 39.37 90)
 			(effects
