File: Sloth/Sloth_panel.kicad_pcb (KiCad board)
At the start: 2 copper layers, 20.3 x 128.5 mm, 0 parts

Commit message: sloth done
Routing:
- added copper zone on F.Cu, net GND
Other:
- board text added: "+"
- board text added: "-"
- board text added: "CV In"
- board text added: "Sloth"
- board text added: "X"
- board text added: "Y"
