File: Sloth/Sloth_torpor.kicad_sch (KiCad schematic)
At the start: 42 parts, among them J1 Out Y, J2 Out X, J3 CV In, J4 Eurorack_Power_10pin_Unshroud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, U1 TL074

Commit message: sloth torpor added
Parts:
- removed C8: 10u, Capacitor_SMD:C_0805_2012Metric_Pad1.18x1.45mm_HandSolder, symbol Device:C
- R1: value 6M8 -> 1M
- R3, R4: value 1M -> 100k
- R6: value 560k -> 100k
- R7: value 10M -> 0
- RV1: value 100k -> 10k
Other:
- note added: "Torpor"
- note removed: "Apathy"
