File: Sloth/Sloth.kicad_sch (KiCad schematic)
At the start: 42 parts, among them J1 Out Y, J2 Out X, J3 CV In, J4 Eurorack_Power_10pin_Unshroud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, U1 TL074

Commit message: added some 3d models and backlog
Parts:
- C4: value 10u -> 1u
- R1: value 6M8 -> 1M
- R3, R4: value 1M -> 100k
- R6: value 560k -> 120k
- R7: value 10M -> 0
- V1: value 12 -> 11.8
- V2: value 12 -> 10.8
Connections:
- net at D1.2 (A), D2.1 (K): no longer R14.2
- net at D3.1 (K), D4.2 (A): no longer R13.2
Changed lines of the file:
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@@
 	)
 	(junction
-		(at 139.7 120.65)
-		(diameter 0)
-		(color 0 0 0 0)
-	)
-	(junction
 		(at 31.75 111.76)
 		(diameter 0)
@@
 	(wire
 		(pts
-			(xy 31.75 92.71) (xy 40.64 92.71)
-		)
-		(stroke
-			(width 0)
-			(type default)
-		)
-	)
-	(wire
-		(pts
 			(xy 69.85 110.49) (xy 64.77 110.49)
 		)
@@
 	(wire
 		(pts
-			(xy 139.7 120.65) (xy 139.7 106.68)
-		)
-		(stroke
-			(width 0)
-			(type default)
-		)
-	)
-	(wire
-		(pts
 			(xy 85.09 163.83) (xy 85.09 161.29)
 		)
@@
 	(wire
 		(pts
-			(xy 139.7 120.65) (xy 143.51 120.65)
+			(xy 135.89 120.65) (xy 143.51 120.65)
 		)
 		(stroke
@@
 	(wire
 		(pts
-			(xy 135.89 120.65) (xy 139.7 120.65)
-		)
-		(stroke
-			(width 0)
-			(type default)
-		)
-	)
-	(wire
-		(pts
 			(xy 116.84 163.83) (xy 119.38 163.83)
 		)
@@
 			)
 		)
-		(property "Value" "10M"
+		(property "Value" "0"
 			(at 52.07 38.1 90)
 			(effects
@@
 		(at 119.38 171.45 0)
 		(unit 1)
-		(exclude_from_sim no)
+		(exclude_from_sim yes)
 		(in_bom yes)
 		(on_board yes)
@@
 			)
 		)
-		(property "Value" "6M8"
+		(property "Value" "1M"
 			(at 54.61 21.59 90)
 			(effects
@@
 			)
 		)
-		(property "Value" "10u"
+		(property "Value" "1u"
 			(at 86.36 115.5699 0)
 			(effects
@@
 			)
 		)
-		(property "Value" "560k"
+		(property "Value" "120k"
 			(at 59.69 55.88 90)
 			(effects
@@
 			)
 		)
-		(property "Value" "12"
+		(property "Value" "11.8"
 			(at 60.96 167.7697 0)
 			(effects
@@
 			)
 		)
-		(property "Value" "12"
+		(property "Value" "10.8"
 			(at 43.18 167.5101 0)
 			(effects
@@
 			)
 		)
-		(property "Value" "1M"
+		(property "Value" "100k"
 			(at 92.71 83.82 90)
 			(effects
@@
 			)
 		)
-		(property "Value" "1M"
+		(property "Value" "100k"
 			(at 73.66 83.82 90)
 			(effects
@@
 		(at 119.38 166.37 0)
 		(unit 1)
-		(exclude_from_sim no)
+		(exclude_from_sim yes)
 		(in_bom yes)
 		(on_board yes)
@@
 			)
 		)
-		(property "Sim.Params" "r=100k"
+		(property "Sim.Params" "r=0"
 			(at 82.55 71.12 0)
 			(effects
