File: splt_mlt/splt_mlt.kicad_pcb (KiCad board)
At the start: 2 copper layers, 26 x 110 mm, 53 parts, among them J1 AudioJack3_SwitchT, J10 AudioJack3_SwitchT, J11 AudioJack3_SwitchT, J12 AudioJack3_SwitchT, J13 AudioJack3_SwitchT, J14 AudioJack3_SwitchT, J15 AudioJack3_SwitchT, J16 AudioJack3_SwitchT, J17 AudioJack3_SwitchT, J2 PWR, J3 AudioJack3_SwitchT, J4 AudioJack3_SwitchT, J5 AudioJack3_SwitchT, J6 AudioJack3_SwitchT, J7 AudioJack3_SwitchT, J8 AudioJack3_SwitchT, J9 AudioJack3_SwitchT, U1 TL074, U2 TL074

Commit message: pltmlt gerbers
Connections:
- J12 pad TN: unconnected-(J12-PadTN) -> Net-(J12-PadTN)
- J13 pad T: Net-(J13-PadT) -> Net-(J12-PadTN)
- J13 pad TN: unconnected-(J13-PadTN) -> Net-(J12-PadT)
- J14 pad TN: unconnected-(J14-PadTN) -> Net-(J14-PadTN)
- J15 pad T: Net-(J15-PadT) -> Net-(J14-PadTN)
- J15 pad TN: unconnected-(J15-PadTN) -> Net-(J14-PadT)
- J16 pad R: Net-(J13-PadT) -> Net-(J12-PadTN)
- J17 pad R: Net-(J15-PadT) -> Net-(J14-PadTN)
Routing:
- net Net-(J14-PadTN): track 0.00 -> 56.3 mm
- net Net-(J15-PadT): track 37.6 -> 0.00 mm
- net Net-(J12-PadTN): track 0.00 -> 35.2 mm
- net Net-(J13-PadT): track 33.7 -> 0.00 mm
- net Net-(J14-PadT): track 15.5 -> 26.1 mm
- net Net-(J12-PadT): track 15.5 -> 22.2 mm
- net Net-(J11-PadT): track 0.00 -> 4.46 mm
- net Net-(D1-A): track 73.0 -> 71.2 mm
