File: splt_mlt/splt_mlt.kicad_sch (KiCad schematic)
At the start: 25 parts, among them J1 AudioJack3_SwitchT, J10 AudioJack3_SwitchT, J2 AudioJack3_SwitchT, J3 Conn_02x05_Counter_Clockwise, J4 AudioJack3_SwitchT, J5 AudioJack3_SwitchT, J7 AudioJack3_SwitchT, J8 AudioJack3_SwitchT, J9 AudioJack3_SwitchT, U1 TL074

Commit message: splt schematic, pcb done
Parts:
- removed J3: Conn_02x05_Counter_Clockwise, symbol Connector_Generic:Conn_02x05_Counter_Clockwise
- removed R1: R_Small, symbol Device:R_Small
- added C1, C2, C7: 100n, Capacitor_SMD:C_0805_2012Metric_Pad1.18x1.45mm_HandSolder, symbol Device:C_Small
- added C10, C11, C12, C9: 1n, Capacitor_SMD:C_0805_2012Metric_Pad1.18x1.45mm_HandSolder, symbol Device:C_Small
- added C13, C14: 10u, Capacitor_THT:CP_Radial_D4.0mm_P1.50mm, symbol Device:C_Polarized_Small
- added D1, D2: 1N5819, Diode_THT:D_DO-41_SOD81_P2.54mm_Vertical_AnodeUp, symbol Device:D_Small
- added J10, J11, J14, J15, J17, J7, J8, J9: AudioJack3_SwitchT, mort_mix:CLIFF_FC681374V, symbol Connector_Audio:AudioJack3_SwitchT
- added J2: PWR, mort_mix:Pins_2x05_2.54mm_TH_Europower_shrouded, symbol Connector_Generic:Conn_02x05_Odd_Even
- added R10, R11, R12, R13, R14, R15, R16, R17, R18: 0, Resistor_SMD:R_0805_2012Metric_Pad1.20x1.40mm_HandSolder, symbol Device:R_Small
- added U2: TL074, Package_SO:SO-14_3.9x8.65mm_P1.27mm, symbol Amplifier_Operational:TL074
- C3: renamed from C2; footprint (none) -> Capacitor_SMD:C_0805_2012Metric_Pad1.18x1.45mm_HandSolder
- C4, C5: footprint (none) -> Capacitor_SMD:C_0805_2012Metric_Pad1.18x1.45mm_HandSolder
- C6: renamed from C3; footprint (none) -> Capacitor_SMD:C_0805_2012Metric_Pad1.18x1.45mm_HandSolder
- C8: renamed from C1; value C_Small -> 100n; footprint (none) -> Capacitor_SMD:C_0805_2012Metric_Pad1.18x1.45mm_HandSolder
- R1: renamed from R6; value 20k -> 0; footprint (none) -> Resistor_SMD:R_0805_2012Metric_Pad1.20x1.40mm_HandSolder
- R2: value 1k -> 0; footprint (none) -> Resistor_SMD:R_0805_2012Metric_Pad1.20x1.40mm_HandSolder
- R3: renamed from R4; value 1k -> 0; footprint (none) -> Resistor_SMD:R_0805_2012Metric_Pad1.20x1.40mm_HandSolder
- R4: renamed from R5; value 1k -> 0; footprint (none) -> Resistor_SMD:R_0805_2012Metric_Pad1.20x1.40mm_HandSolder
- R5: renamed from R3; value 1k -> 0; footprint (none) -> Resistor_SMD:R_0805_2012Metric_Pad1.20x1.40mm_HandSolder
- R6: renamed from R7; value 100 -> 0; footprint (none) -> Resistor_SMD:R_0805_2012Metric_Pad1.20x1.40mm_HandSolder
- R7: renamed from R8; value 100 -> 0; footprint (none) -> Resistor_SMD:R_0805_2012Metric_Pad1.20x1.40mm_HandSolder
- R8: renamed from R9; value 100 -> 0; footprint (none) -> Resistor_SMD:R_0805_2012Metric_Pad1.20x1.40mm_HandSolder
- R9: renamed from R10; value 100 -> 0; footprint (none) -> Resistor_SMD:R_0805_2012Metric_Pad1.20x1.40mm_HandSolder
- U1: footprint (none) -> Package_SO:SO-14_3.9x8.65mm_P1.27mm
- renumbered J8 to J1, J1 to J12, J9 to J13, J7 to J16, J10 to J3, J2 to J4, J4 to J5, J5 to J6
Connections:
- net GND: now also C8.2, J1.TN, C1.1, C13.1, C14.2, C2.2, C7.1, J10.S, J11.S, J14.S, J15.S, J17.S, J2.3 (Pin_3), J2.4 (Pin_4), J2.5 (Pin_5), J2.6 (Pin_6), J2.7 (Pin_7), J2.8 (Pin_8), J7.S, J8.S, J9.S
- net at R1.2, U1.10 (+), U1.12 (+)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: now also J7.TN
- net at C8.1: now also U1.4 (V+), C14.1, C2.1, D2.1 (K), U2.4 (V+)
- net at U1.11 (V-): now also C1.2, C13.2, C7.2, D1.2 (A), U2.11 (V-)
- new net: C10.1, R12.1, U2.6 (-)
- new net: C10.2, R12.2, R16.1, U2.7
- new net: D1.1 (K), J2.1 (Pin_1), J2.2 (Pin_2)
- new net: D2.2 (A), J2.10 (Pin_10), J2.9 (Pin_9)
- new net: R10.2, U2.10 (+), U2.12 (+), U2.3 (+), U2.5 (+)
- new net: C12.1, R14.1, U2.13 (-)
- new net: C12.2, R14.2, R18.1, U2.14
- new net: C11.2, R13.2, R17.1, U2.8
- new net: C11.1, R13.1, U2.9 (-)
- new net: J8.T, R15.2
- new net: J15.T, J17.R
- new net: J14.T, J17.T
- new net: J7.T, R10.1
- new net: C9.2, R11.2, R15.1, U2.1
- new net: C9.1, R11.1, U2.2 (-)
- new net: J10.T, R17.2
- new net: J11.T, R18.2
- new net: J9.T, R16.2
- no-connect marks 15 -> 28
Other:
- moved on the sheet: C8, J12, J13, J16, U1E

Commit message: pltmlt gerbers
Connections:
- net at J13.T, J16.R: now also J12.TN
- net at J13.TN: now also J12.T, J16.T
- net at J15.T, J17.R: now also J14.TN
- net at J14.T, J17.T: now also J15.TN
- no-connect marks 28 -> 24
Changed lines of the file:
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@@
+	)
+	(junction
+		(at 245.11 90.17)
+		(diameter 0)
+		(color 0 0 0 0)
 	)
 	(junction
@@
 	)
 	(junction
+		(at 245.11 38.1)
+		(diameter 0)
+		(color 0 0 0 0)
+	)
+	(junction
 		(at 57.15 114.3)
 		(diameter 0)
@@
 	)
 	(junction
+		(at 248.92 43.18)
+		(diameter 0)
+		(color 0 0 0 0)
+	)
+	(junction
 		(at 50.8 175.26)
 		(diameter 0)
@@
 	)
 	(junction
+		(at 248.92 95.25)
+		(diameter 0)
+		(color 0 0 0 0)
+	)
+	(junction
 		(at 83.82 182.88)
 		(diameter 0)
@@
 	)
 	(no_connect
-		(at 241.3 92.71)
-	)
-	(no_connect
 		(at 193.04 123.19)
 	)
@@
 	)
 	(no_connect
-		(at 241.3 40.64)
-	)
-	(no_connect
 		(at 86.36 118.11)
 	)
@@
 	)
 	(no_connect
-		(at 241.3 64.77)
-	)
-	(no_connect
 		(at 86.36 74.93)
 	)
 	(no_connect
-		(at 241.3 116.84)
-	)
-	(no_connect
 		(at 193.04 90.17)
 	)
@@
 	(wire
 		(pts
+			(xy 245.11 38.1) (xy 257.81 38.1)
+		)
+		(stroke
+			(width 0)
+			(type default)
+		)
+	)
+	(wire
+		(pts
+			(xy 241.3 40.64) (xy 248.92 40.64)
+		)
+		(stroke
+			(width 0)
+			(type default)
+		)
+	)
+	(wire
+		(pts
 			(xy 163.83 77.47) (xy 168.91 77.47)
 		)
@@
 	(wire
 		(pts
+			(xy 241.3 116.84) (xy 245.11 116.84)
+		)
+		(stroke
+			(width 0)
+			(type default)
+		)
+	)
+	(wire
+		(pts
 			(xy 189.23 92.71) (xy 193.04 92.71)
 		)
@@
 	(wire
 		(pts
+			(xy 245.11 90.17) (xy 257.81 90.17)
+		)
+		(stroke
+			(width 0)
+			(type default)
+		)
+	)
+	(wire
+		(pts
+			(xy 245.11 64.77) (xy 245.11 38.1)
+		)
+		(stroke
+			(width 0)
+			(type default)
+		)
+	)
+	(wire
+		(pts
 			(xy 57.15 41.91) (xy 57.15 38.1)
 		)
@@
 	(wire
 		(pts
+			(xy 241.3 64.77) (xy 245.11 64.77)
+		)
+		(stroke
+			(width 0)
+			(type default)
+		)
+	)
+	(wire
+		(pts
 			(xy 241.3 62.23) (xy 248.92 62.23)
 		)
@@
 	(wire
 		(pts
-			(xy 241.3 38.1) (xy 257.81 38.1)
+			(xy 241.3 38.1) (xy 245.11 38.1)
 		)
 		(stroke
@@
 	(wire
 		(pts
+			(xy 248.92 40.64) (xy 248.92 43.18)
+		)
+		(stroke
+			(width 0)
+			(type default)
+		)
+	)
+	(wire
+		(pts
 			(xy 72.39 38.1) (xy 72.39 44.45)
 		)
@@
 	(wire
 		(pts
+			(xy 248.92 92.71) (xy 248.92 95.25)
+		)
+		(stroke
+			(width 0)
+			(type default)
+		)
+	)
+	(wire
+		(pts
 			(xy 46.99 72.39) (xy 46.99 97.79)
 		)
@@
 	(wire
 		(pts
-			(xy 241.3 90.17) (xy 257.81 90.17)
+			(xy 241.3 90.17) (xy 245.11 90.17)
 		)
 		(stroke
@@
 		)
 		(stroke
+			(width 0)
+			(type default)
+		)
+	)
+	(wire
+		(pts
+			(xy 241.3 92.71) (xy 248.92 92.71)
+		)
+		(stroke
+			(width 0)
+			(type default)
+		)
+	)
+	(wire
+		(pts
+			(xy 245.11 116.84) (xy 245.11 90.17)
+		)
+		(stroke
