File: templates/templates.kicad_pcb (KiCad board)
At the start: 2 copper layers, 180.2 x 128.5 mm, 0 parts

Commit message: daisy patch.init
Routing:
- net (no net): vias 16 -> 17
Other:
- board text added: "Pushbutton Switch"
- board text removed: "Mounting Hole"
Changed lines of the file:
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@@
 	)
 	(gr_text "Poti"
-		(at 80.64 189.75 0)
-		(layer "User.6")
-		(effects
-			(font
-				(size 1 1)
-				(thickness 0.15)
-			)
-		)
-	)
-	(gr_text "Mounting Hole"
-		(at 118.64 189.75 0)
-		(layer "User.6")
-		(effects
-			(font
-				(size 1 1)
-				(thickness 0.15)
-			)
+		(at 86.64 189.75 0)
+		(layer "User.6")
+		(effects
+			(font
+				(size 1 1)
+				(thickness 0.15)
+			)
+			(justify top)
 		)
 	)
@@
 				(thickness 0.15)
 			)
+			(justify top)
 		)
 	)
 	(gr_text "LED"
-		(at 118.64 191.75 0)
-		(layer "User.6")
-		(effects
-			(font
-				(size 1 1)
-				(thickness 0.15)
-			)
+		(at 126.64 189.75 0)
+		(layer "User.6")
+		(effects
+			(font
+				(size 1 1)
+				(thickness 0.15)
+			)
+			(justify top)
 		)
 	)
@@
 		)
 	)
+	(gr_text "Pushbutton\nSwitch\n"
+		(at 116.64 189.75 0)
+		(layer "User.6")
+		(effects
+			(font
+				(size 1 1)
+				(thickness 0.15)
+			)
+			(justify top)
+		)
+	)
 	(gr_text "4HP\n"
 		(at 44.64 29.75 0)
@@
 	)
 	(gr_text "MiniSwitch"
-		(at 92.64 189.75 0)
-		(layer "User.6")
-		(effects
-			(font
-				(size 1 1)
-				(thickness 0.15)
-			)
+		(at 96.64 189.75 0)
+		(layer "User.6")
+		(effects
+			(font
+				(size 1 1)
+				(thickness 0.15)
+			)
+			(justify top)
 		)
 	)
@@
 	)
 	(via
+		(at 116.64 183.75)
+		(size 5)
+		(drill 4)
+		(layers "F.Cu" "B.Cu")
+		(net 0)
+	)
+	(via
 		(at 43.26 39.75)
 		(size 4)
@@
 	)
 	(via
-		(at 92.64 183.75)
+		(at 96.64 183.75)
 		(size 7.5)
 		(drill 6.5)
@@
 	)
 	(via
-		(at 118.640002 183.75)
+		(at 126.64 183.75)
 		(size 4)
 		(drill 3)
@@
 	)
 	(via
-		(at 80.64 183.75)
+		(at 86.64 183.75)
 		(size 8)
 		(drill 7)
