File: Teletype/teletype-180824_1.kicad_sch (KiCad schematic)
At the start: 74 parts, among them IC2 OKI-78SR, J40 ISP-ROW, SW40 PANASONIC-EVQ, U1 TPS2021, U2 AT32UC3B064/0128/0256, U3 AD5687R, U4 AD5687R, U40 ADP3339, U44 BAS70-04, U6 BAS70-04, U7 AD7923, X1 2510-, Y1 12mhz

Commit message: working on teletype
Parts:
- removed C1, C18, C26, C27, C29, C3, C30, C31, C41, C42, C46, C47, C50, C56, C59, C7: 100n, Teletype:C0402, symbol Teletype-eagle-import:C_0402
- removed C10, C12, C16, C17, C45, C52, C53, C54: 33n, Teletype:C0402, symbol Teletype-eagle-import:C_0402
- removed C11: 470p, Teletype:C0402, symbol Teletype-eagle-import:C_0402
- removed C13, C14, C15, C8: 2.7n, Teletype:C0402, symbol Teletype-eagle-import:C_0402
- removed C19, C20: 22p, Teletype:C0402, symbol Teletype-eagle-import:C_0402
- removed C2: 220u, Teletype:C7343-43, symbol Teletype-eagle-import:CP_7343-43
- removed C24, C25, C28, C4, C44, C6, C60: 10u, Teletype:C1206_T, symbol Teletype-eagle-import:CP_1206/T
- removed C48, C55, C9: 2.2u, Teletype:C0603, symbol Teletype-eagle-import:C_0603
- removed C49, C51: 4.7u, Teletype:C0603, symbol Teletype-eagle-import:C_0603
- removed C5: 4.7u, Teletype:C1206_T, symbol Teletype-eagle-import:CP_1206/T
- removed IC2: OKI-78SR, Teletype:TO220V, symbol Teletype-eagle-import:78TV
- removed J40: ISP-ROW, Teletype:ISP-ROW, symbol Teletype-eagle-import:ISP-ROW
- removed JP1, JP2: PINHD-2X3, Teletype:2X03, symbol Teletype-eagle-import:PINHD-2X3
- removed PF1, PF2: PTC-F0805-15V, Teletype:F1206, symbol Teletype-eagle-import:PTC-F1206
- removed R1, R2: 47k, Teletype:R0402, symbol Teletype-eagle-import:R_0402
- removed R16, R5: 2k, Teletype:R0402, symbol Teletype-eagle-import:R_0402
- removed R4, R40: 10k, Teletype:R0402, symbol Teletype-eagle-import:R_0402
- removed R41, R42, R48: 0, Teletype:R0402, symbol Teletype-eagle-import:R_0402
- removed R43, R44: 39, Teletype:R0402, symbol Teletype-eagle-import:R_0402
- removed R45: 0, Teletype:R0603, symbol Teletype-eagle-import:R_0603
- removed SW40: PANASONIC-EVQ, Teletype:PANASONIC-EVQ, symbol Teletype-eagle-import:PANASONIC-EVQ
- removed U1: TPS2021, Teletype:SO08, symbol Teletype-eagle-import:TPS2020
- removed U2: AT32UC3B064/0128/0256, Teletype:TQFP64-10X10, symbol Teletype-eagle-import:AT32UC3B064/0128/0256
- removed U3, U4: AD5687R, Teletype:TSSOP16, symbol Teletype-eagle-import:AD5689R
- removed U40: ADP3339, Teletype:SOT223, symbol Teletype-eagle-import:ADP3339
- removed U44, U6: BAS70-04, Teletype:SOT23, symbol Teletype-eagle-import:BAS70-04
- removed U7: AD7923, Teletype:TSSOP16, symbol Teletype-eagle-import:AD7923
- removed X1: 2510-, Teletype:PAK100_2500-10, symbol Teletype-eagle-import:2510-
- removed Y1: 12mhz, Teletype:HC49UP, symbol Teletype-eagle-import:CRYTALHC49UP
- added C1, C18, C26, C27, C29, C3, C30, C31, C41, C42, C46, C47, C50, C56, C59, C7: 100n, teletype-180824:C0402, symbol teletype-180824-eagle-import:C_0402
- added C10, C12, C16, C17, C45, C52, C53, C54: 33n, teletype-180824:C0402, symbol teletype-180824-eagle-import:C_0402
- added C11: 470p, teletype-180824:C0402, symbol teletype-180824-eagle-import:C_0402
- added C13, C14, C15, C8: 2.7n, teletype-180824:C0402, symbol teletype-180824-eagle-import:C_0402
- added C19, C20: 22p, teletype-180824:C0402, symbol teletype-180824-eagle-import:C_0402
- added C2: 220u, teletype-180824:C7343-43, symbol teletype-180824-eagle-import:CP_7343-43
- added C24, C25, C28, C4, C44, C6, C60: 10u, teletype-180824:C1206_T, symbol teletype-180824-eagle-import:CP_1206/T
- added C48, C55, C9: 2.2u, teletype-180824:C0603, symbol teletype-180824-eagle-import:C_0603
- added C49, C51: 4.7u, teletype-180824:C0603, symbol teletype-180824-eagle-import:C_0603
- added C5: 4.7u, teletype-180824:C1206_T, symbol teletype-180824-eagle-import:CP_1206/T
- added IC2: OKI-78SR, teletype-180824:TO220V, symbol teletype-180824-eagle-import:78TV
- added J40: ISP-ROW, teletype-180824:ISP-ROW, symbol teletype-180824-eagle-import:ISP-ROW
- added JP1, JP2: PINHD-2X3, teletype-180824:2X03, symbol teletype-180824-eagle-import:PINHD-2X3
- added PF1, PF2: PTC-F0805-15V, teletype-180824:F1206, symbol teletype-180824-eagle-import:PTC-F1206
- added R1, R2: 47k, teletype-180824:R0402, symbol teletype-180824-eagle-import:R_0402
- added R16, R5: 2k, teletype-180824:R0402, symbol teletype-180824-eagle-import:R_0402
- added R4, R40: 10k, teletype-180824:R0402, symbol teletype-180824-eagle-import:R_0402
- added R41, R42, R48: 0, teletype-180824:R0402, symbol teletype-180824-eagle-import:R_0402
- added R43, R44: 39, teletype-180824:R0402, symbol teletype-180824-eagle-import:R_0402
- added R45: 0, teletype-180824:R0603, symbol teletype-180824-eagle-import:R_0603
- added SW40: PANASONIC-EVQ, teletype-180824:PANASONIC-EVQ, symbol teletype-180824-eagle-import:PANASONIC-EVQ
- added U1: TPS2021, teletype-180824:SO08, symbol teletype-180824-eagle-import:TPS2020
- added U2: AT32UC3B064/0128/0256, teletype-180824:TQFP64-10X10, symbol teletype-180824-eagle-import:AT32UC3B064/0128/0256
- added U3, U4: AD5687R, teletype-180824:TSSOP16, symbol teletype-180824-eagle-import:AD5689R
- added U40: ADP3339, teletype-180824:SOT223, symbol teletype-180824-eagle-import:ADP3339
- added U44, U6: BAS70-04, teletype-180824:SOT23, symbol teletype-180824-eagle-import:BAS70-04
- added U7: AD7923, teletype-180824:TSSOP16, symbol teletype-180824-eagle-import:AD7923
- added X1: 2510-, teletype-180824:PAK100_2500-10, symbol teletype-180824-eagle-import:2510-
- added Y1: 12mhz, teletype-180824:HC49UP, symbol teletype-180824-eagle-import:CRYTALHC49UP
Connections:
- net +12V: now also C3.2, C6.+, IC2.1 (VI), PF2.1, PF2.2, U6.2 (C2), X1.10 (KL), X1.9 (KL)
- net +3V3: now also C24.+, C25.+, C26.2, C27.2, C28.+, C29.2, C30.2, C44.+, R16.2, R4.2, R40.2, R41.2, R42.2, R5.2, U2.18 (ADVREF), U2.19 (VDDANA), U3.11 (VLOGIC), U3.15 (_RESET), U3.5 (VDD), U4.11 (VLOGIC), U4.15 (_RESET), U4.5 (VDD), U40.2 (OUT), U40.4 (OUTP), U44.2 (C2), U7.15 (VDRIVE), U7.5 (AVDD), U7.6 (AVDD2)
- net +5V: now also C2.+, C42.2, C59.2, C60.+, IC2.3 (VO), R1.2, R2.2, U1.2 (IN1), U1.3 (IN2), U40.3 (IN)
- net -12V: now also C1.2, C4.-, PF1.1, PF1.2, U6.1 (A1), X1.1 (KL), X1.2 (KL)
- net A00: now also U2.3 (TDI/GPIO0)
- net A01: now also U2.4 (TDO/GPIO1)
- net A02: now also U2.5 (TMS/GPIO2)
- net A03: now also U2.9 (PA03/GPIO3/ADC0/GCLK0/USB_ID)
- net A04: now also U2.10 (PA04/GPIO4/ADC1/USB_VBOF)
- net A05: now also U2.11 (PA05/GPIO5/EXTINT0/ADC2/USART1-DCD)
- net A06: now also U2.12 (PA06/GPIO6/ADC3/USART1-DSR)
- net A07: now also U2.13 (PA07/GPIO7/PWM0/ADC4/USART1-DTR)
- net AGND: now also C24.-, C25.-, C26.1, C27.1, C28.-, C29.1, C30.1, R45.1, U3.10 (GAIN), U3.16 (RSTSEL), U3.4 (GND), U3.9 (_LDAC), U4.10 (GAIN), U4.16 (RSTSEL), U4.4 (GND), U4.9 (_LDAC), U44.1 (A1), U7.10 (VIN2), U7.13 (AGND3), U7.16 (AGND4), U7.4 (AGND), U7.8 (AGND2), U7.9 (VIN3)
- net B08: now also U2.54 (PB08/GPIO40/SSC-RX_FRAME_SYNC/USART1-DTR/EIC-SCAN6)
- net B09: now also U2.55 (PB09/GPIO41/SSC-TX_CLOCK/USART1-RI/EIC-SCAN7)
- net B10: now also U2.57 (PB10/GPIO42/SSC-TX_DATA/TC-A2/USART0-RXD)
- net B11: now also U2.58 (PB11/GPIO43/SSC-TX_FRAME_SYNC/TC-B2/USART0-TXD)
- net CS0: now also U2.36 (PA16/GPIO16/SPI-CS0/TC-CLK1), U3.13 (_SYNC), U4.13 (_SYNC)
- net CS1: now also U2.37 (PA17/GPIO17/SPI-CS1/TC-CLK2/SPI-SCK), U7.3 (_CS)
- net CS2: now also U2.27 (PB05/GPIO37/USART1-RTS/SPI-CS2/PWM5)
- net CV-IN0: now also U44.3 (C1A2), U7.12 (VIN0)
- net CV-IN1: now also U7.11 (VIN1)
- net CV-OUT0: now also U3.3 (VOUTA)
- net CV-OUT1: now also U3.7 (VOUTB)
- net CV-OUT2: now also U4.3 (VOUTA)
- net CV-OUT3: now also U4.7 (VOUTB)
- net DM: now also R44.2
- net DP: now also R43.2
- net GND: now also C1.1, C10.1, C11.1, C12.1, C13.1, C14.1, C15.1, C16.1, C17.1, C18.1, C19.1, C2.-, C20.1, C3.1, C31.2, C4.+, C41.2, C42.1, C44.-, C45.1, C46.1, C47.1, C48.1, C49.1, C5.-, C50.1, C51.1, C52.1, C53.1, C54.1, C55.1, C56.1, C59.1, C6.-, C60.-, C7.1, C8.1, C9.1, IC2.2 (GND), J40.1 (VCC), J40.2 (MOSI), JP1.5, JP1.6, JP2.5, JP2.6, R45.2, SW40.1, U1.1 (GND), U2.1 (GND@1), U2.17 (GND@17), U2.23 (GND@23), U2.49 (GND@49), U2.61 (PA26/GPIO26/USB_ID/USART2-TXD/TC-A0), U6.3 (C1A2), X1.3 (KL), X1.4 (KL), X1.5 (KL), X1.6 (KL), X1.7 (KL), X1.8 (KL)
- net MISO: now also U2.41 (PA28/GPIO28/USART0-CLK/PWM4/SPI-MISO/XIN1), U7.14 (DOUT)
- net MOSI: now also U2.42 (PA29/GPIO29/TC-CLK0/TC-CLK1/SPI-MOSI/XOUT1), U3.14 (SDIN), U7.2 (DIN)
- net NMI: now also C31.1, R4.1, U2.33 (PA13/GPIO13/NMI/PWM2/USART0-CLK)
- net OLED-DC: now also U2.26 (PB04/GPIO36/USART1-CTS/SPI-CS3/TC-CLK2)
- net OLED-RES: now also U2.25 (PB03/GPIO35/EXTINT7/TC-B1/USART1-RXD)
- net RX: now also J40.4 (SCK), U2.59 (PA24/GPIO24/USART1-RXD/SPIC-CS0/EXTINT4)
- net SCK: now also U2.35 (PA15/GPIO15/SPI-SCK/PWM4/USART2-CLK), U3.12 (SCLK), U4.12 (SCLK), U7.1 (SCLK)
- net SCL: now also JP1.3, JP1.4, JP2.3, JP2.4, R16.1, U2.28 (PA09/GPIO9/SCL/SPI-CS2/USART1-CTS)
- net SDA: now also JP1.1, JP1.2, JP2.1, JP2.2, R5.1, U2.29 (PA10/GPIO10/SDA/SI-CS3/USART1-RTS)
- net TX: now also J40.5 (RESET), U2.47 (PA23/GPIO23/USART1-TXD/SPI-CS1/EXTIN3)
- net USB-OC: now also R2.1, U1.5 (_OC), U2.60 (PA25/GPIO25/SPI-MISO/PWM3/EXTINT5)
- net USB-VBOF: now also R1.1, U1.4 (_EN), U2.62 (PA27/GPIO27/USB_VBOF/USART2-RXD/TC-B0)
- net VBUS: now also C5.+, C7.2, U1.6 (OUT1), U1.7 (OUT2), U1.8 (OUT3), U2.52 (VBUS)
- net VDDIN: now also C12.2, C50.2, C51.2, R42.1, U2.21 (VDDIN)
- net VDDIO: now also C10.2, C16.2, C17.2, C18.2, C47.2, C49.2, C56.2, R41.1, U2.32 (VDDIO@32), U2.48 (VDDIO@48), U2.64 (VDDIO@64)
- net VDDOUT: now also C11.2, C13.2, C14.2, C15.2, C45.2, C46.2, C48.2, C52.2, C53.2, C54.2, C55.2, C8.2, C9.2, U2.20 (VDDOUT), U2.22 (VDDCORE@22), U2.53 (VDDPLL), U2.56 (VDDCORE@56), U2.8 (VDDCORE@8)
- net VREF: now also U3.1 (VREF), U7.7 (REF)
- new net: R44.1, U2.51 (USB_DM)
- new net: C19.2, U2.40 (PA19/GPIO19/USART0-TXD/PWM6/SPI-MOSI/XOUT), Y1.1
- new net: R43.1, U2.50 (USB_DP)
- new net: C20.2, U2.39 (PA18/GPIO18/USART0-RXD/PWM5/SPI-MISO/XIN), Y1.2
- new net: R48.1, U2.6 (PB00/GPIO32/TC-A0/EIC-SCAN2/USART2-CTS)
- new net: R48.2, U2.7 (PB01/GPIO33/TC-B0/EIC-SCAN3/USART2-RTS)
- new net: C41.1, R40.1, SW40.2, U2.63 (~{RESET})
- new net: U3.8 (SDO), U4.14 (SDIN)
