File: Teletype/teletype-180824_2.kicad_sch (KiCad schematic)
At the start: 98 parts, among them IC1 TL074, IC4 OPA4171, J1 WQP-PJ301M-12_JACK, J10 WQP-PJ301M-12_JACK, J11 WQP-PJ301M-12_JACK, J12 WQP-PJ301M-12_JACK, J13 WQP-PJ301M-12_JACK, J14 WQP-PJ301M-12_JACK, J15 WQP-PJ301M-12_JACK, J16 WQP-PJ301M-12_JACK, J17 WQP-PJ301M-12_JACK, J2 WQP-PJ301M-12_JACK, J3 WQP-PJ301M-12_JACK, J4 WQP-PJ301M-12_JACK, J5 WQP-PJ301M-12_JACK, J6 WQP-PJ301M-12_JACK, J7 WQP-PJ301M-12_JACK, J8 WQP-PJ301M-12_JACK, J9 WQP-PJ301M-12_JACK, P1 10k

Commit message: working on teletype
Parts:
- removed C21, C22, C23, C32: 100n, Teletype:C0402, symbol Teletype-eagle-import:C-USC0402
- removed C33: 33n, Teletype:C0402, symbol Teletype-eagle-import:C-USC0402
- removed C34, C35, C36, C37, C38, C39, C43, C57, C58: 1n, Teletype:C0402, symbol Teletype-eagle-import:C-USC0402
- removed D2, D3, D4, D5, D6, D7, D8, D9: BAS70-04, Teletype:SOT23, symbol Teletype-eagle-import:BAS70-04
- removed IC1: TL074, Teletype:SO14, symbol Teletype-eagle-import:AD8644R
- removed IC4: OPA4171, Teletype:SO14, symbol Teletype-eagle-import:AD8644R
- removed J1, J10, J11, J12, J13, J14, J15, J16, J17, J2, J3, J4, J5, J6, J7, J8, J9: WQP-PJ301M-12_JACK, Teletype:WQP-PJ301M-12_JACK, symbol Teletype-eagle-import:WQP-PJ301M-12_JACK
- removed LED1, LED2, LED3, LED4: OR, Teletype:CHIP-LED0805, symbol Teletype-eagle-import:LEDCHIP-LED0805
- removed LED5, LED6, LED7, LED8: W, Teletype:CHIP-LED0805, symbol Teletype-eagle-import:LEDCHIP-LED0805
- removed P1: 10k, Teletype:SHAPES_POT-ALPS_ALPS_POT_VERTICAL_PS, symbol Teletype-eagle-import:SHAPES_POT-ALPS_POT_USVERTICAL_PS
- removed POP0: SWITCH-OMRON_10-XX, Teletype:SWITCH-OMRON_B3F-10XX, symbol Teletype-eagle-import:SWITCH-OMRON_10-XX
- removed R10, R14, R17, R21, R29, R3, R51, R8: 1k, Teletype:R0402, symbol Teletype-eagle-import:R-US_R0402
- removed R11, R12, R13, R18, R22, R26, R28, R31, R33, R35, R39, R6, R7, R9: 10k, Teletype:R0402, symbol Teletype-eagle-import:R-US_R0402
- removed R15, R19, R23, R24, R25, R27, R30, R32, R34, R36, R56, R58, R60: 30k, Teletype:R0402, symbol Teletype-eagle-import:R-US_R0402
- removed R20: 31k6, Teletype:R0402, symbol Teletype-eagle-import:R-US_R0402
- removed R37, R38, R46, R47, R52, R53, R66, R67: 20k, Teletype:R0402, symbol Teletype-eagle-import:R-US_R0402
- removed RN1: 47k, Teletype:MNR35, symbol Teletype-eagle-import:RESNET08
- removed U$1: OLED128X64, Teletype:OLED-ALEPH, symbol Teletype-eagle-import:OLED128X64
- removed USB0: SHAPES_PONY_MOLEX-USB-VERT, Teletype:SHAPES_PONY_MOLEX-USB, symbol Teletype-eagle-import:SHAPES_PONY_MOLEX-USB-VERT
- added C21, C22, C23, C32: 100n, teletype-180824:C0402, symbol teletype-180824-eagle-import:C-USC0402
- added C33: 33n, teletype-180824:C0402, symbol teletype-180824-eagle-import:C-USC0402
- added C34, C35, C36, C37, C38, C39, C43, C57, C58: 1n, teletype-180824:C0402, symbol teletype-180824-eagle-import:C-USC0402
- added D2, D3, D4, D5, D6, D7, D8, D9: BAS70-04, teletype-180824:SOT23, symbol teletype-180824-eagle-import:BAS70-04
- added IC1: TL074, teletype-180824:SO14, symbol teletype-180824-eagle-import:AD8644R
- added IC4: OPA4171, teletype-180824:SO14, symbol teletype-180824-eagle-import:AD8644R
- added J1, J10, J11, J12, J13, J14, J15, J16, J17, J2, J3, J4, J5, J6, J7, J8, J9: WQP-PJ301M-12_JACK, teletype-180824:WQP-PJ301M-12_JACK, symbol teletype-180824-eagle-import:WQP-PJ301M-12_JACK
- added LED1, LED2, LED3, LED4: OR, teletype-180824:CHIP-LED0805, symbol teletype-180824-eagle-import:LEDCHIP-LED0805
- added LED5, LED6, LED7, LED8: W, teletype-180824:CHIP-LED0805, symbol teletype-180824-eagle-import:LEDCHIP-LED0805
- added P1: 10k, teletype-180824:SHAPES_POT-ALPS_ALPS_POT_VERTICAL_PS, symbol teletype-180824-eagle-import:SHAPES_POT-ALPS_POT_USVERTICAL_PS
- added POP0: SWITCH-OMRON_10-XX, teletype-180824:SWITCH-OMRON_B3F-10XX, symbol teletype-180824-eagle-import:SWITCH-OMRON_10-XX
- added R10, R14, R17, R21, R29, R3, R51, R8: 1k, teletype-180824:R0402, symbol teletype-180824-eagle-import:R-US_R0402
- added R11, R12, R13, R18, R22, R26, R28, R31, R33, R35, R39, R6, R7, R9: 10k, teletype-180824:R0402, symbol teletype-180824-eagle-import:R-US_R0402
- added R15, R19, R23, R24, R25, R27, R30, R32, R34, R36, R56, R58, R60: 30k, teletype-180824:R0402, symbol teletype-180824-eagle-import:R-US_R0402
- added R20: 31k6, teletype-180824:R0402, symbol teletype-180824-eagle-import:R-US_R0402
- added R37, R38, R46, R47, R52, R53, R66, R67: 20k, teletype-180824:R0402, symbol teletype-180824-eagle-import:R-US_R0402
- added RN1: 47k, teletype-180824:MNR35, symbol teletype-180824-eagle-import:RESNET08
- added U$1: OLED128X64, teletype-180824:OLED-ALEPH, symbol teletype-180824-eagle-import:OLED128X64
- added USB0: SHAPES_PONY_MOLEX-USB-VERT, teletype-180824:SHAPES_PONY_MOLEX-USB, symbol teletype-180824-eagle-import:SHAPES_PONY_MOLEX-USB-VERT
Connections:
- net +12V: now also C21.1, C23.1, IC1.4 (V+), IC4.4 (V+)
- net +3V3: now also D2.2 (C2), D3.2 (C2), D4.2 (C2), D5.2 (C2), D6.2 (C2), D7.2 (C2), D8.2 (C2), D9.2 (C2), P1.P$1 (E), U$1.2 (VDD)
- net -12V: now also C22.2, C32.2, IC1.11 (V-), IC4.11 (V-)
- net A00: now also C37.1, D3.3 (C1A2), R32.2, RN1.7 (6)
- net A01: now also C35.1, D2.3 (C1A2), R27.2, RN1.5
- net A02: now also C36.1, D4.3 (C1A2), R30.2, RN1.8 (7)
- net A03: now also C38.1, D5.3 (C1A2), R34.2, RN1.4
- net A04: now also C39.1, D6.3 (C1A2), R36.2, RN1.9 (8)
- net A05: now also C43.1, D7.3 (C1A2), R56.2, RN1.3
- net A06: now also C57.1, D8.3 (C1A2), R58.2, RN1.10 (9)
- net A07: now also C58.1, D9.3 (C1A2), R60.2, RN1.2
- net AGND: now also C33.2, C34.2, P1.P$3 (A), R20.2, R26.1
- net B08: now also IC1.5 (IN+)
- net B09: now also IC1.3 (IN+)
- net B10: now also IC1.12 (IN+)
- net B11: now also IC1.10 (IN+)
- net CS2: now also U$1.17 (/CS)
- net CV-IN0: now also C34.1, R24.2, R26.2
- net CV-IN1: now also C33.1, R18.2, R20.1
- net CV-OUT0: now also IC4.3 (IN+)
- net CV-OUT1: now also IC4.5 (IN+)
- net CV-OUT2: now also IC4.10 (IN+)
- net CV-OUT3: now also IC4.12 (IN+)
- net DM: now also USB0.2
- net DP: now also USB0.3
- net GND: now also C21.2, C22.1, C23.2, C32.1, C35.2, C36.2, C37.2, C38.2, C39.2, C43.2, C57.2, C58.2, D2.1 (A1), D3.1 (A1), D4.1 (A1), D5.1 (A1), D6.1 (A1), D7.1 (A1), D8.1 (A1), D9.1 (A1), J1.SLEEVE, J10.SLEEVE, J11.SLEEVE, J12.SLEEVE, J13.SLEEVE, J14.SLEEVE, J15.SLEEVE, J16.SLEEVE, J17.SLEEVE, J17.TS, J2.SLEEVE, J3.SLEEVE, J4.SLEEVE, J5.SLEEVE, J6.SLEEVE, J7.SLEEVE, J8.SLEEVE, J9.SLEEVE, LED1.C, LED2.C, LED3.C, LED4.C, LED5.C, LED6.C, LED7.C, LED8.C, POP0.3 (P), POP0.4 (P1), R12.1, R13.1, R22.1, R28.1, R31.1, R33.1, R35.1, R39.1, RN1.1, RN1.6 (10), U$1.1 (VSS), U$1.10 (DB3), U$1.11 (DB4), U$1.12 (DB5), U$1.13 (DB6), U$1.14 (DB7), U$1.19 (BS1), U$1.20 (BS0), U$1.5 (R/W), U$1.6 (E), U$1.9 (DB2), USB0.GND, USB0.M1 (S1), USB0.M2 (S1), USB0.M4 (S1)
- net MOSI: now also U$1.8 (SDIN)
- net NMI: now also POP0.1 (S), POP0.2 (S1)
- net OLED-DC: now also U$1.4 (D/C)
- net OLED-RES: now also U$1.16 (/RES)
- net SCK: now also U$1.7 (SCLK)
- net VBUS: now also USB0.1
- new net: J6.TIP, R56.1
- new net: IC1.13 (IN-), R22.2, R46.1
- new net: IC1.14 (OUT), R14.1, R46.2, R9.1
- new net: IC4.6 (IN-), R25.1, R33.2
- new net: J14.TIP, R25.2, R29.2
- new net: LED3.A, R9.2
- new net: IC1.9 (IN-), R28.2, R47.1
- new net: IC1.8 (OUT), R10.1, R11.1, R47.2
- new net: IC4.14 (OUT), R51.1, R53.1
- new net: LED8.A, R53.2
- new net: J1.TIP, R32.1
- new net: P1.P$2 (S), R18.1
- new net: IC4.13 (IN-), R23.1, R39.2
- new net: IC4.9 (IN-), R15.1, R35.2
- new net: IC1.6 (IN-), R12.2, R38.1
- new net: IC1.7 (OUT), R3.1, R38.2, R6.1
- new net: J2.TIP, R27.1
- new net: J16.TIP, R23.2, R51.2
- new net: LED7.A, R52.2
- new net: J7.TIP, R58.1
- new net: IC4.8 (OUT), R17.1, R52.1
- new net: J15.TIP, R15.2, R17.2
- new net: J11.TIP, R14.2
- new net: IC4.7 (OUT), R29.1, R67.1
- new net: LED2.A, R7.2
- new net: LED4.A, R11.2
- new net: J5.TIP, R36.1
- new net: LED5.A, R66.2
- new net: J9.TIP, R3.2
- new net: J17.TIP, R24.1
- new net: IC4.2 (IN-), R19.1, R31.2
- new net: J3.TIP, R30.1
- new net: J8.TIP, R60.1
- new net: J12.TIP, R10.2
- new net: LED6.A, R67.2
- new net: LED1.A, R6.2
- new net: IC1.2 (IN-), R13.2, R37.1
- new net: IC1.1 (OUT), R37.2, R7.1, R8.1
- new net: J13.TIP, R19.2, R21.2
- new net: J10.TIP, R8.2
- new net: IC4.1 (OUT), R21.1, R66.1
- new net: J4.TIP, R34.1
- no-connect marks 0 -> 16
