File: Teletype/teletype-180824.kicad_pcb (KiCad board)
At the start: 4 copper layers, 88.9 x 109.9 mm, 172 parts, among them IC1 TL074, IC2 OKI-78SR, IC4 OPA4171, J1 WQP-PJ301M-12_JACK, J10 WQP-PJ301M-12_JACK, J11 WQP-PJ301M-12_JACK, J12 WQP-PJ301M-12_JACK, J13 WQP-PJ301M-12_JACK, J14 WQP-PJ301M-12_JACK, J15 WQP-PJ301M-12_JACK, J16 WQP-PJ301M-12_JACK, J17 WQP-PJ301M-12_JACK, J2 WQP-PJ301M-12_JACK, J3 WQP-PJ301M-12_JACK, J4 WQP-PJ301M-12_JACK, J40 ISP-ROW, J5 WQP-PJ301M-12_JACK, J6 WQP-PJ301M-12_JACK, J7 WQP-PJ301M-12_JACK, J8 WQP-PJ301M-12_JACK, J9 WQP-PJ301M-12_JACK, P1 10k, SW40 PANASONIC-EVQ, U1 TPS2021, U2 AT32UC3B064/0128/0256, U3 AD5687R, U4 AD5687R, U40 ADP3339, U44 BAS70-04, U6 BAS70-04, U7 AD7923, X1 2510-, Y1 12mhz

Commit message: added some 3d models and backlog
Other:
- board text added: "Clandestine Circutry Console"
- board text removed: "monome.org teletype180824"
