File: elements/hardware_design/pcb/KiCad/elements_v02_1.kicad_sch (KiCad schematic)
At the start: 36 parts, among them IC10 STM32F405RGT6, IC12 WM8731, Q1 8MHz, SW2 EVQQ2, SW3 EVQQ2

Commit message: Marbles added
Beware! T_clock is shorted to ground. Fix before using this PCB
Parts:
- C52: footprint elements_v02:PANASONIC_B -> Capacitor_SMD:CP_Elec_6.3x5.4
