File: elements/hardware_design/pcb/KiCad/elements_v02_2.kicad_sch (KiCad schematic)
At the start: 27 parts, among them IC14 LME49720, J5 PJ301_THONKICONN6, J6 PJ301_THONKICONN6, J7 PJ301_THONKICONN6, J8 PJ301_THONKICONN6

Commit message: Marbles added
Beware! T_clock is shorted to ground. Fix before using this PCB
Parts:
- C40, C53, C55, C56: footprint elements_v02:PANASONIC_B -> Capacitor_SMD:CP_Elec_6.3x5.4
