File: elements/hardware_design/pcb/KiCad/elements_v02_5.kicad_sch (KiCad schematic)
At the start: 19 parts, among them IC1 LM4040B10, IC2 LM1117-3.3, IC4 LM1117-3.3

Commit message: Marbles added
Beware! T_clock is shorted to ground. Fix before using this PCB
Parts:
- C1, C10, C3, C9: footprint elements_v02:PANASONIC_C -> Capacitor_SMD:CP_Elec_6.3x5.9
